File: SMT_Soldering_class.kicad_pcb (KiCad board)
At the start: 2 copper layers, 59 parts, among them J1 AVR-ISP-6, J2 USB_B_Micro, J3 Conn_01x04, U1 ATmega48PB-A, Y1 16MHz

Commit message: version 1.0, march 2023, ready to fab
Parts:
- removed C3: 100nF, Capacitor_SMD:C_0805_2012Metric_Pad1.18x1.45mm_HandSolder
- removed C5: 22pF, Capacitor_SMD:C_0805_2012Metric_Pad1.18x1.45mm_HandSolder
- removed Y1: 16MHz, Crystal:Crystal_SMD_ECS_CSM3X-2Pin_7.6x4.1mm
- added kibuzzard-6403760C: G***, kibuzzard-6403760C, F.Cu at (105.4, 104.4)
- added kibuzzard-64037C19: G***, kibuzzard-64037C19, F.Cu at (122.4, 95.5)
- added kibuzzard-64037C58: G***, kibuzzard-64037C58, F.Cu at (88.4, 104.6)
- added kibuzzard-64037C81: G***, kibuzzard-64037C81, F.Cu at (145.8, 109.2)
- added kibuzzard-64037CBD: G***, kibuzzard-64037CBD, F.Cu at (127.3, 108.5)
- added kibuzzard-64037CBD: G***, kibuzzard-64037CBD, F.Cu at (85.1, 110.5)
- added kibuzzard-6404A9BB: G***, kibuzzard-6404A9BB, B.Cu at (121.2, 94.2)
- C4: value 22pF -> 4.7uF
- moved R1 83.0 mm to (131.6, 108.0)
- moved C4 82.5 mm to (135.1, 102.9), turned to 90 degrees
- moved C2 81.1 mm to (131.6, 102.9), turned to -90 degrees
- moved J3 73.8 mm to (101.6, 110.7), turned to 90 degrees
- moved J2 68.1 mm to (155.2, 109.7)
- moved C1 63.0 mm to (112.8, 101.9), turned to -90 degrees
- moved U1 58.9 mm to (122.1, 103.8)
- moved D1 55.3 mm to (91.8, 101.5)
- moved D10 55.3 mm to (128.8, 80.1)
- moved R11 55.3 mm to (130.7, 73.8)
- moved R12 55.3 mm to (136.8, 76.0)
- moved R13 55.3 mm to (142.3, 79.2)
- moved R14 55.3 mm to (147.2, 83.3)
- moved R17 55.3 mm to (156.8, 99.8)
- moved TP1 55.3 mm to (96.7, 102.8)
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Connections:
- C4 pad 1: Net-(C4-Pad1) -> VCC
- U1 pad 28: /LED1 -> /LED0
- U1 pad 32: /LED0 -> /LED1
- U1 pad 7: Net-(C4-Pad1) -> unconnected-(U1-Pad7)
- U1 pad 8: Net-(C5-Pad1) -> unconnected-(U1-Pad8)
Routing:
- net VCC: track 98.9 -> 184.9 mm, vias 0 -> 2
- net /RESET: track 0.00 -> 41.9 mm, vias 0 -> 3
- net /SDI: track 0.00 -> 41.3 mm, vias 0 -> 1
- net /SDO: track 0.00 -> 41.2 mm, vias 0 -> 1
- net /SCK: track 0.00 -> 35.8 mm, vias 0 -> 2
- net /LED1: track 4.05 -> 37.3 mm
- net /LED0: track 4.05 -> 33.9 mm
- net /LED2: track 4.04 -> 32.1 mm
- net /LED3: track 4.03 -> 31.8 mm
- net /LED4: track 4.01 -> 29.8 mm
- net /LED5: track 3.98 -> 26.2 mm
- net /LED13: track 3.71 -> 25.8 mm
- net /LED12: track 0.00 -> 21.1 mm
- net /LED15: track 3.66 -> 24.6 mm
- net /LED14: track 3.68 -> 24.5 mm
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- added copper zone on B.Cu, net GND
Other:
- board outline added: 79.2 x 43.4 mm
