File: SMT_Soldering_class.kicad_sch (KiCad schematic)
At the start: 11 parts, among them J1 AVR-ISP-6, J2 USB_B_Micro, J3 Conn_01x04, U1 ATmega48PB-A, Y1 16MHz

Commit message: version 1.0, march 2023, ready to fab
Parts:
- removed C3: 100nF, Capacitor_SMD:C_0805_2012Metric_Pad1.18x1.45mm_HandSolder, symbol Device:C
- removed C5: 22pF, Capacitor_SMD:C_0805_2012Metric_Pad1.18x1.45mm_HandSolder, symbol Device:C
- removed Y1: 16MHz, Crystal:Crystal_SMD_ECS_CSM3X-2Pin_7.6x4.1mm, symbol Device:Crystal
- C4: value 22pF -> 4.7uF
Connections:
- net LED0: now also U1.28 (PC5); no longer U1.32 (PD2)
- net LED1: now also U1.32 (PD2); no longer U1.28 (PC5)
- net VCC: now also C4.1
- net at U1.7 (XTAL1/PB6): no longer C4.1
- no-connect marks 5 -> 7
