File: led.kicad_sch (KiCad schematic)
At the start: 3 parts

Commit message: version 1.0, march 2023, ready to fab
Parts:
- renumbered D1 to D16, R2 to R17, TP1 to TP16
Changed lines of the file:
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@@
   (symbol (lib_id "Connector:TestPoint") (at 137.795 107.315 90)
     (in_bom yes) (on_board yes) (fields_autoplaced)
-    (property "Reference" "TP1" (id 0) (at 134.493 101.6 90))
+    (property "Reference" "TP16" (id 0) (at 134.493 101.6 90))
     (property "Value" "TestPoint" (id 1) (at 134.493 104.14 90))
     (property "Footprint" "TestPoint:TestPoint_Pad_D2.0mm" (id 2) (at 137.795 102.235 0)
@@
   (symbol (lib_id "Device:LED") (at 137.795 96.52 90)
     (in_bom yes) (on_board yes) (fields_autoplaced)
-    (property "Reference" "D1" (id 0) (at 140.97 96.8374 90)
+    (property "Reference" "D16" (id 0) (at 140.97 96.8374 90)
       (effects (font (size 1.27 1.27)) (justify right))
     )
@@
   (symbol (lib_id "power:VCC") (at 137.795 79.375 0)
     (in_bom yes) (on_board yes) (fields_autoplaced)
-    (property "Reference" "#PWR014" (id 0) (at 137.795 83.185 0)
+    (property "Reference" "#PWR029" (id 0) (at 137.795 83.185 0)
       (effects (font (size 1.27 1.27)) hide)
     )
@@
   (symbol (lib_id "Device:R") (at 137.795 85.725 0)
     (in_bom yes) (on_board yes) (fields_autoplaced)
-    (property "Reference" "R2" (id 0) (at 139.7 84.4549 0)
+    (property "Reference" "R17" (id 0) (at 139.7 84.4549 0)
       (effects (font (size 1.27 1.27)) (justify left))
     )
