File: VU_board/board/SMT_Soldering_class.kicad_pcb (KiCad board)
At the start: 2 copper layers, 79.2 x 43.4 mm, 63 parts, among them J1 AVR-ISP-6, J2 USB_B_Micro, J3 Conn_01x04, U1 ATmega48PB-A

Commit message: added switch to PCB adding modes to firmware (for old version)
Parts:
- removed kibuzzard-6404A9BB: G***, kibuzzard-6404A9BB
- added SW1: SW_Push, Button_Switch_SMD:SW_Push_1P1T-SH_NO_CK_KMR2xxG, F.Cu at (137.9, 110.1)
- added kibuzzard-6419EFEB: G***, kibuzzard-6419EFEB, B.Cu at (121.7, 94.2)
- added kibuzzard-641A1732: G***, kibuzzard-641A1732, F.Cu at (145.0, 109.5)
- moved kibuzzard-64037C81 10.3 mm to (155.3, 105.3)
Connections:
- U1 pad 7: unconnected-(U1-Pad7) -> Net-(U1-Pad7)
Routing:
- net Net-(U1-Pad7): track 0.00 -> 19.5 mm, vias 0 -> 2
- net GND: track 20.7 -> 25.6 mm, vias 5 -> 6
- net /LED11: track 21.2 -> 19.2 mm
