File: VU_board/board/led.kicad_sch (KiCad schematic)
At the start: 3 parts

Commit message: added switch to PCB adding modes to firmware (for old version)
Other:
- company: (none) -> NYC Resistor
- title: (none) -> LED block
Changed lines of the file:
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@@
 (kicad_sch (version 20211123) (generator eeschema)
   (paper "A4")
+  (title_block
+    (title "LED block")
+    (rev "v1")
+    (company "NYC Resistor")
+  )
   (junction (at 137.795 107.315) (diameter 0) (color 0 0 0 0)
   )
